Commit message: fix(urdf): 修正 LiDAR 安裝朝向為反裝 180 度
實測 LiDAR 將正前方 0.26m 的牆面回報在 180 度、而正前方回報
1.86m 淨空，確認其 0 度指向車體後方，但 URDF 與 tf_config 都
假設 rpy 為零。

base_link->laser 缺少這 180 度會讓 SLAM 與 AMCL 的航向估計整整
差 180 度：前端圖示前後顛倒、實際後退顯示為前進，且 scan matching
會持續與里程計衝突，此前建立的地圖均無效。

新增 properties.xacro 的 laser_yaw 參數集中管理，tf_config.yaml
的 fallback 路徑同步修正。

另補回 meshes/ 目錄佔位檔——該目錄為空而未被 git 追蹤，遺失後
CMakeLists 的 install(DIRECTORY meshes) 會導致建置失敗。

File: src/robot_description/urdf/properties.xacro (robot description, xacro)
@@ -30,5 +30,8 @@
   <xacro:property name="laser_x" value="0.0"/>             <!-- 前方 0cm -->
   <xacro:property name="laser_y" value="0.0"/>             <!-- 中心 -->
-  <xacro:property name="laser_z" value="0.336"/>            <!-- 高度 40cm -->
+  <xacro:property name="laser_z" value="0.336"/>            <!-- 高度 33.6cm -->
+  <!-- LiDAR 安裝朝向（繞 z 軸，弧度）。實體反裝故為 pi；
+       若日後改為正裝請改回 0，並同步 motor_control/config/tf_config.yaml -->
+  <xacro:property name="laser_yaw" value="${pi}"/>
   <!-- ========== IMU 感測器位置 ========== -->
   <!-- 相對於 base_link -->

File: src/robot_description/urdf/robot.urdf.xacro (robot description, xacro)
@@ -161,5 +161,7 @@
     <parent link="base_link"/>
     <child link="laser"/>
-    <origin xyz="${laser_x} ${laser_y} ${laser_z}" rpy="0 0 0"/>
+    <!-- LiDAR 實體反裝：其 0° 指向車體後方，故需繞 z 軸旋轉 180°。
+         漏掉這個旋轉會讓 SLAM/AMCL 的航向估計整整差 180 度。 -->
+    <origin xyz="${laser_x} ${laser_y} ${laser_z}" rpy="0 0 ${laser_yaw}"/>
   </joint>
   <link name="laser">

Commit message: fix(motor): 重校有效輪距 0.27 -> 0.3514
舊值 0.27 是在驅動器磁極對數設錯（設 5、實際 4）時代校的，
吸收了 RPM 回報 x0.8 的尺度誤差；驅動器極對數修正後旋轉
odom 多報 30%（單圈 1.307、雙圈 1.3016 兩次實測互證）。

以 720 度旋轉測試重校：0.27 x 1.3016 = 0.3514（有效輪距，
含原地旋轉打滑效應）。同步 hs_motor_config、properties.xacro、
bringup mock 參數與 mock 預設值，避免模擬與真機分岔。

File: src/robot_description/urdf/properties.xacro (robot description, xacro)
@@ -9,5 +9,5 @@
   <!-- ========== 輪子參數 ========== -->
   <!-- 來源: motor_control/config/hs_motor_config.yaml -->
-  <xacro:property name="wheel_separation" value="0.27"/>   <!-- 輪距 (m) -->
+  <xacro:property name="wheel_separation" value="0.3514"/>   <!-- 有效輪距 (m)，2026-07-24 旋轉校正，與 hs_motor_config.yaml 同步 -->
   <xacro:property name="wheel_radius" value="0.065"/>      <!-- 輪半徑 (m) -->
   <xacro:property name="wheel_width" value="0.032"/>        <!-- 輪寬 (m) -->
